Commit message: remove code so it renders in colab?

File: assets/descriptions/bittle/urdf/bittle.urdf (robot description, URDF)
Before this commit: robot bittle, 13 links, 12 joints
Links:
- link base-frame-link: geometry collision mesh filename=assets/descriptions/bittle/meshes/obj/base_frame.001.obj scale=1.0 1.0 1.0; visual mesh filename=assets/descriptions/bittle/meshes/obj/base_frame.obj scale=1.0 1.0 1.0
- link battery-link: geometry collision mesh filename=assets/descriptions/bittle/meshes/obj/battery.001.obj scale=1.0 1.0 1.0; visual mesh filename=assets/descriptions/bittle/meshes/obj/battery.obj scale=1.0 1.0 1.0
- link cover-link: geometry collision mesh filename=assets/descriptions/bittle/meshes/obj/cover.001.obj scale=1.0 1.0 1.0; visual mesh filename=assets/descriptions/bittle/meshes/obj/cover.obj scale=1.0 1.0 1.0
- link imu_link: geometry visual mesh filename=assets/descriptions/bittle/meshes/obj/Cube.011.obj scale=1.0 1.0 1.0
- link left-back-knee-link: geometry collision mesh filename=assets/descriptions/bittle/meshes/obj/left_knee.002.obj scale=1.0 1.0 1.0; visual mesh filename=assets/descriptions/bittle/meshes/obj/left_knee.001.obj scale=1.0 1.0 1.0
- link left-back-shoulder-link: geometry collision mesh filename=assets/descriptions/bittle/meshes/obj/shoulder.004.obj scale=1.0 1.0 1.0; visual mesh filename=assets/descriptions/bittle/meshes/obj/shoulder.001.obj scale=1.0 1.0 1.0
- link left-front-knee-link: geometry collision mesh filename=assets/descriptions/bittle/meshes/obj/left_knee.003.obj scale=1.0 1.0 1.0; visual mesh filename=assets/descriptions/bittle/meshes/obj/left_knee.obj scale=1.0 1.0 1.0
- link left-front-shoulder-link: geometry collision mesh filename=assets/descriptions/bittle/meshes/obj/shoulder.007.obj scale=1.0 1.0 1.0; visual mesh filename=assets/descriptions/bittle/meshes/obj/shoulder.obj scale=1.0 1.0 1.0
- link mainboard_link: geometry visual mesh filename=assets/descriptions/bittle/meshes/obj/Plane.obj scale=1.0 1.0 1.0
- link right-back-knee-link: geometry collision mesh filename=assets/descriptions/bittle/meshes/obj/right_knee.002.obj scale=1.0 1.0 1.0; visual mesh filename=assets/descriptions/bittle/meshes/obj/right_knee.001.obj scale=1.0 1.0 1.0
- link right-back-shoulder-link: geometry collision mesh filename=assets/descriptions/bittle/meshes/obj/shoulder.005.obj scale=1.0 1.0 1.0; visual mesh filename=assets/descriptions/bittle/meshes/obj/shoulder.002.obj scale=1.0 1.0 1.0
- link right-front-knee-link: geometry collision mesh filename=assets/descriptions/bittle/meshes/obj/right_knee.003.obj scale=1.0 1.0 1.0; visual mesh filename=assets/descriptions/bittle/meshes/obj/right_knee.obj scale=1.0 1.0 1.0
- link right-front-shoulder-link: geometry collision mesh filename=assets/descriptions/bittle/meshes/obj/shoulder.006.obj scale=1.0 1.0 1.0; visual mesh filename=assets/descriptions/bittle/meshes/obj/shoulder.003.obj scale=1.0 1.0 1.0

Commit message: added mujoco extension to urdf file and converted successfully to mjcf

File: assets/descriptions/bittle/urdf/bittle.urdf (robot description, URDF)
Before this commit: robot bittle, 13 links, 12 joints
Links:
- link base-frame-link: geometry collision mesh filename=base_frame.001.obj scale=1.0 1.0 1.0; visual mesh filename=base_frame.obj scale=1.0 1.0 1.0
- link battery-link: geometry collision mesh filename=battery.001.obj scale=1.0 1.0 1.0; visual mesh filename=battery.obj scale=1.0 1.0 1.0
- link cover-link: geometry collision mesh filename=cover.001.obj scale=1.0 1.0 1.0; visual mesh filename=cover.obj scale=1.0 1.0 1.0
- link imu_link: geometry visual mesh filename=Cube.011.obj scale=1.0 1.0 1.0
- link left-back-knee-link: geometry collision mesh filename=left_knee.002.obj scale=1.0 1.0 1.0; visual mesh filename=left_knee.001.obj scale=1.0 1.0 1.0
- link left-back-shoulder-link: geometry collision mesh filename=shoulder.004.obj scale=1.0 1.0 1.0; visual mesh filename=shoulder.001.obj scale=1.0 1.0 1.0
- link left-front-knee-link: geometry collision mesh filename=left_knee.003.obj scale=1.0 1.0 1.0; visual mesh filename=left_knee.obj scale=1.0 1.0 1.0
- link left-front-shoulder-link: geometry collision mesh filename=shoulder.007.obj scale=1.0 1.0 1.0; visual mesh filename=shoulder.obj scale=1.0 1.0 1.0
- link mainboard_link: geometry visual mesh filename=Plane.obj scale=1.0 1.0 1.0
- link right-back-knee-link: geometry collision mesh filename=right_knee.002.obj scale=1.0 1.0 1.0; visual mesh filename=right_knee.001.obj scale=1.0 1.0 1.0
- link right-back-shoulder-link: geometry collision mesh filename=shoulder.005.obj scale=1.0 1.0 1.0; visual mesh filename=shoulder.002.obj scale=1.0 1.0 1.0
- link right-front-knee-link: geometry collision mesh filename=right_knee.003.obj scale=1.0 1.0 1.0; visual mesh filename=right_knee.obj scale=1.0 1.0 1.0
- link right-front-shoulder-link: geometry collision mesh filename=shoulder.006.obj scale=1.0 1.0 1.0; visual mesh filename=shoulder.003.obj scale=1.0 1.0 1.0
